File: pcb/passthrough.kicad_pcb (KiCad board)
At the start: 2 copper layers, 13 x 36 mm, 13 parts

Commit message: Add license information to many files. PCB design files are CC-BY and code is MIT license.
Other:
- board text added: "Copyright 2016 Chickadee Tech LLC, <add attributions here> This work is licensed under the Creative Commons Attribution 4.0 International License. To view a copy of this license, visit http://creativecommons.org/licenses/by/4.0/ or send a letter to Creative Commons, PO Box 1866, Mountain View, CA 94042, USA."
- board text added: "Remove all Chickadee Tech LLC trademarks before making your own board. The Chickadee logo and Polystack logo are owned by Chickadee Tech LLC. You may license the Polystack logo for free by emailing support@chickadee.tech and receiving express written permission from Chickadee Tech LLC."
Changed lines of the file:
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@@
-(kicad_pcb (version 4) (host pcbnew "(2015-11-03 BZR 6296)-product")
+(kicad_pcb (version 4) (host pcbnew 4.0.1-stable)
   (general
-    (links 0)
+    (links 123)
     (no_connects 0)
-    (area 118.127143 74.1 233.214289 178)
+    (area 152.924999 89.924999 166.075001 126.075001)
     (thickness 1.6)
-    (drawings 25)
+    (drawings 28)
     (tracks 841)
     (zones 0)
@@
       (xy -2.200426 -1.477507) (xy -2.158969 -1.476897)) (layer F.Mask) (width 0.01))
   )
+  (gr_text "Copyright 2016 Chickadee Tech LLC, <add attributions here>\n\nThis work is licensed under the Creative Commons Attribution 4.0 International License.\nTo view a copy of this license, visit http://creativecommons.org/licenses/by/4.0/\nor send a letter to Creative Commons, PO Box 1866, Mountain View, CA 94042, USA." (at 178.06 173.82) (layer Cmts.User)
+    (effects (font (size 1.5 1.5) (thickness 0.3)) (justify left))
+  )
+  (gr_line (start 152.84 122.54) (end 133.67 130.73) (layer Cmts.User) (width 0.2))
+  (gr_text "Remove all Chickadee Tech LLC trademarks\nbefore making your own board. The\nChickadee logo and Polystack logo\nare owned by Chickadee Tech LLC.\n\nYou may license the Polystack logo for\nfree by emailing support@chickadee.tech\nand receiving express written permission\nfrom Chickadee Tech LLC." (at 93.47 132.59) (layer Cmts.User)
+    (effects (font (size 1.5 1.5) (thickness 0.3)) (justify left))
+  )
   (gr_text ckd.tech/pt/v1 (at 159.56 118.76) (layer B.SilkS)
     (effects (font (size 1 1) (thickness 0.15)) (justify mirror))
@@
   (gr_line (start 166 92.75) (end 166 123.25) (angle 90) (layer Edge.Cuts) (width 0.15))
   (gr_line (start 154 90) (end 163.25 90) (angle 90) (layer Edge.Cuts) (width 0.15))
-  (gr_text passthrough (at 187.25 174.25) (layer Cmts.User)
-    (effects (font (size 5 5) (thickness 0.5)) (justify left))
+  (gr_text passthrough (at 186.76 189.45) (layer Cmts.User)
+    (effects (font (size 3 3) (thickness 0.5)) (justify left))
   )
   (segment (start 162.95 97.849974) (end 162.95 96.45) (width 0.1524) (layer F.Cu) (net 1))
